File: hardware/GB-v2-87L/GB-v2-87L.kicad_pcb (KiCad board)
At the start: 2 copper layers, 196 x 35 mm, 90 parts, among them J1 Conn_01x02

Commit message: - Introduced a new footprint for a 2.7mm mounting hole in the ProjectSpecific library. - Updated schematic references to use the new footprint instead of the previous generic mounting hole.
Parts:
- H1, H2: footprint MountingHole:MountingHole_2.7mm_M2.5_DIN965_Pad -> ProjectSpecific:MountingHole_2.7mm
Routing:
- net Net-(D22-K): track 8.64 -> 0.00 mm
