File: hardware/GB-v2-87L/GB-v2-87L.kicad_sch (KiCad schematic)
At the start: 90 parts, among them J1 Conn_01x02

Commit message: - Introduced a new footprint for a 2.7mm mounting hole in the ProjectSpecific library. - Updated schematic references to use the new footprint instead of the previous generic mounting hole.
Parts:
- H1, H2: footprint MountingHole:MountingHole_2.7mm_M2.5_DIN965_Pad -> ProjectSpecific:MountingHole_2.7mm
Changed lines of the file:
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@@
 			)
 		)
-		(property "Footprint" "MountingHole:MountingHole_2.7mm_M2.5_DIN965_Pad"
+		(property "Footprint" "ProjectSpecific:MountingHole_2.7mm"
 			(at 207.01 66.04 0)
 			(effects
@@
 			)
 		)
-		(property "Footprint" "MountingHole:MountingHole_2.7mm_M2.5_DIN965_Pad"
+		(property "Footprint" "ProjectSpecific:MountingHole_2.7mm"
 			(at 207.01 58.42 0)
 			(effects
